Commit message: gz

File: my_first_car/urdf/robot.urdf.xacro (robot description, xacro)
@@ -7,4 +7,46 @@
     <color rgba="0.1 0.1 0.1 1.0"/>
 </material>
+<xacro:property name="wheel_radius" value="0.05"/>
+<xacro:property name="wheel_length" value="0.04"/>
+<xacro:property name="wheel_mass" value="0.2"/>
+<xacro:property name="base_mass" value="2.0"/>
+<xacro:property name="base_length" value="0.4"/>
+<xacro:property name="base_width" value="0.2"/>
+<xacro:property name="base_height" value="0.1"/>
+<xacro:property name="caster_mass" value="0.1"/>
+<xacro:property name="caster_radius" value="0.03"/>
+<xacro:macro name="wheel" params="prefix y_pos">
+    <link name="${prefix}_wheel">
+        <visual>
+            <geometry>
+                <cylinder radius="${wheel_radius}" length="${wheel_length}"/>
+            </geometry>
+            <origin xyz="0 0 0" rpy="0 0 0"/>
+            <material name="dark"/>
+        </visual>
+        <collision>
+            <geometry>
+                <cylinder radius="${wheel_radius}" length="${wheel_length}"/>
+            </geometry>
+            <origin xyz="0 0 0" rpy="0 0 0"/>
+        </collision>
+        <inertial>
+            <origin xyz="0 0 0" rpy="0 0 0"/>
+            <mass value="${wheel_mass}"/>
+            <inertia
+                ixx="${(1/12) * wheel_mass * (3*wheel_radius*wheel_radius + wheel_length*wheel_length)}"
+                ixy="0" ixz="0"
+                iyy="${(1/12) * wheel_mass * (3*wheel_radius*wheel_radius + wheel_length*wheel_length)}"
+                iyz="0"
+                izz="${(wheel_mass * wheel_radius * wheel_radius) / 2}"/>
+        </inertial>
+    </link>
+<joint name="base_${prefix}_wheel_joint" type="continuous">
+    <parent link="base_link"/>
+    <child link="${prefix}_wheel"/>
+    <origin xyz="0.1 ${y_pos} 0" rpy="1.5708 0 0"/>
+    <axis xyz="0 0 -1"/>
+</joint>
+</xacro:macro>
 <!-- LINKS -->
     <link name="base_link">
@@ -16,23 +58,23 @@
             <material name="blue"/>
         </visual>
+        <collision>
+            <geometry>
+                <box size="0.4 0.2 0.1"/>
+            </geometry>
+            <origin xyz="0 0 0.06" rpy="0 0 0"/>
+        </collision>
+        <inertial>
+            <origin xyz="0 0 0.06" rpy="0 0 0"/>
+            <mass value="${base_mass}"/>
+            <inertia
+                ixx="${(1/12) * base_mass * (base_width*base_width + base_height*base_height)}"
+                ixy="0" ixz="0"
+                iyy="${(1/12) * base_mass * (base_length*base_length + base_height*base_height)}"
+                iyz="0"
+                izz="${(1/12) * base_mass * (base_length*base_length + base_width*base_width)}"/>
+        </inertial>
     </link>
-    <link name="left_wheel">
-        <visual>
-            <geometry>
-                <cylinder radius="0.05" length="0.04"/>
-            </geometry>
-            <origin xyz="0 0 0" rpy="0 0 0"/>
-            <material name="dark"/>
-        </visual>
-    </link>
-    <link name="right_wheel">
-        <visual>
-            <geometry>
-                <cylinder radius="0.05" length="0.04"/>
-            </geometry>
-             <origin xyz="0 0 0" rpy="0 0 0"/>
-             <material name="dark"/>
-        </visual>
-    </link>
+<xacro:wheel prefix="left" y_pos="0.12"/>
+<xacro:wheel prefix="right" y_pos="-0.12"/>
     <link name="caster_wheel">
         <visual>
@@ -43,18 +85,22 @@
             <origin xyz="0 0 0" rpy="0 0 0"/>
         </visual>
+        <collision>
+            <geometry>
+                <sphere radius="0.03"/>
+            </geometry>
+            <origin xyz="0 0 0" rpy="0 0 0"/>
+        </collision>
+                <inertial>
+            <origin xyz="0 0 0" rpy="0 0 0"/>
+            <mass value="${caster_mass}"/>
+            <inertia
+                ixx="${(2/5) * caster_mass * caster_radius * caster_radius}"
+                ixy="0" ixz="0"
+                iyy="${(2/5) * caster_mass * caster_radius * caster_radius}"
+                iyz="0"
+                izz="${(2/5) * caster_mass * caster_radius * caster_radius}"/>
+        </inertial>
     </link>
     <!-- JOINTS -->
-<joint name="base_left_wheel_joint" type="continuous">
-    <parent link="base_link"/>
-    <child link="left_wheel"/>
-    <origin xyz="0.1 0.12 0" rpy="1.5708 0 0"/>
-    <axis xyz="0 0 1"/>
-</joint>
-<joint name="base_right_wheel_joint" type="continuous">
-    <parent link="base_link"/>
-    <child link="right_wheel"/>
-    <origin xyz="0.1 -0.12 0" rpy="1.5708 0 0"/>
-    <axis xyz="0 0 1"/>
-</joint>
 <joint name="base_caster_wheel_joint" type="fixed">
     <parent link="base_link"/>
@@ -62,3 +108,16 @@
     <origin xyz="-0.1 0 -0.02" rpy="0 0 0"/>
 </joint>
+<gazebo>
+    <plugin filename="gz-sim-diff-drive-system"
+            name="gz::sim::systems::DiffDrive">
+        <left_joint>base_left_wheel_joint</left_joint>
+        <right_joint>base_right_wheel_joint</right_joint>
+        <wheel_separation>0.24</wheel_separation>
+        <wheel_radius>${wheel_radius}</wheel_radius>
+        <topic>cmd_vel</topic>
+        <odom_publish_frequency>30</odom_publish_frequency>
+        <frame_id>odom</frame_id>
+        <child_frame_id>base_link</child_frame_id>
+    </plugin>
+</gazebo>
 </robot>

Commit message: new project

File: my_first_car/urdf/robot.urdf.xacro (robot description, xacro)
@@ -50,4 +50,11 @@
 </xacro:macro>
 <!-- LINKS -->
+    <link name="base_footprint">
+    </link>
+    <joint name="footprint_link_joint" type="fixed">
+        <parent link="base_footprint"/>
+        <child link="base_link"/>
+        <origin xyz="-0.1 0 0.05" rpy="0 0 0"/>
+    </joint>
     <link name="base_link">
         <visual>
@@ -118,5 +125,5 @@
         <odom_publish_frequency>30</odom_publish_frequency>
         <frame_id>odom</frame_id>
-        <child_frame_id>base_link</child_frame_id>
+        <child_frame_id>base_footprint</child_frame_id>
     </plugin>
 </gazebo>
