Commit message: Add front caster, obstacle avoidance node

File: mybot/urdf/mybot.urdf.xacro (robot description, xacro)
@@ -114,4 +114,24 @@
         </inertial>
     </link>
+        <link name="caster_front">
+        <visual>
+            <geometry>
+                <sphere radius="${caster_radius}"/>
+            </geometry>
+            <origin xyz="0 0 0" rpy="0 0 0"/>
+            <material name="black"></material>
+        </visual>
+        <collision>
+            <geometry>
+                <sphere radius="${caster_radius}"/>
+            </geometry>
+        </collision>
+        <inertial>
+            <mass value="${caster_mass}"/>
+            <inertia ixx="${0.4 * caster_mass * caster_radius * caster_radius}" ixy="0" ixz="0"
+                     iyy="${0.4 * caster_mass * caster_radius * caster_radius}" iyz="0"
+                     izz="${0.4 * caster_mass * caster_radius * caster_radius}"/>
+        </inertial>
+    </link>
     <!-- JOINT -->
     <joint name="base_joint" type="fixed">
@@ -129,4 +149,9 @@
         <child link="lidar_link"/>
         <origin xyz="0 0 0.085" rpy="0 0 0"/>
+    </joint>
+    <joint name="caster_front_joint" type="fixed">
+        <parent link="base_link"/>
+        <child link="caster_front"/>
+        <origin xyz="0.05 0 ${caster_radius - wheel_radius}" rpy="0 0 0"/>
     </joint>
         <!-- ===== Gazebo ===== -->
@@ -178,3 +203,7 @@
         </sensor>
     </gazebo>
+    <gazebo reference="caster_front">
+        <mu1>0.001</mu1>
+        <mu2>0.001</mu2>
+    </gazebo>
 </robot>

Commit message: Add IMU, EKF sensor fusion, joystick teleop and updated map

File: mybot/urdf/mybot.urdf.xacro (robot description, xacro)
@@ -134,4 +134,21 @@
         </inertial>
     </link>
+        <link name="imu_link">
+        <visual>
+            <geometry><box size="0.02 0.02 0.01"/></geometry>
+        </visual>
+        <collision>
+            <geometry><box size="0.02 0.02 0.01"/></geometry>
+        </collision>
+        <inertial>
+            <mass value="0.01"/>
+            <inertia ixx="1e-6" ixy="0" ixz="0" iyy="1e-6" iyz="0" izz="1e-6"/>
+        </inertial>
+    </link>
+    <joint name="imu_joint" type="fixed">
+        <parent link="base_link"/>
+        <child link="imu_link"/>
+        <origin xyz="0 0 0.03" rpy="0 0 0"/>
+    </joint>
     <!-- JOINT -->
     <joint name="base_joint" type="fixed">
@@ -166,5 +183,4 @@
             <frame_id>odom</frame_id>
             <child_frame_id>base_footprint</child_frame_id>
-            <tf_topic>/tf</tf_topic>
             <odom_publisher_frequency>30</odom_publisher_frequency>
         </plugin>
@@ -203,4 +219,21 @@
         </sensor>
     </gazebo>
+        <gazebo reference="imu_link">
+        <sensor name="imu_sensor" type="imu">
+            <always_on>true</always_on>
+            <update_rate>100</update_rate>
+            <topic>imu</topic>
+            <gz_frame_id>imu_link</gz_frame_id>
+            <imu>
+                <angular_velocity>
+                    <z><noise type="gaussian"><mean>0.0</mean><stddev>0.0005</stddev></noise></z>
+                </angular_velocity>
+                <linear_acceleration>
+                    <x><noise type="gaussian"><mean>0.0</mean><stddev>0.01</stddev></noise></x>
+                    <y><noise type="gaussian"><mean>0.0</mean><stddev>0.01</stddev></noise></y>
+                </linear_acceleration>
+            </imu>
+        </sensor>
+    </gazebo>
     <gazebo reference="caster_front">
         <mu1>0.001</mu1>

Commit message: Add camera sensor and bridge

File: mybot/urdf/mybot.urdf.xacro (robot description, xacro)
@@ -22,4 +22,8 @@
     <xacro:property name="caster_mass" value="0.02" />
     <xacro:property name="lidar_mass" value="0.1" />
+    <xacro:property name="cam_x" value="0.03"/>
+    <xacro:property name="cam_y" value="0.08"/>
+    <xacro:property name="cam_z" value="0.03"/>
+    <xacro:property name="cam_mass" value="0.02"/>
     <xacro:macro name="wheel" params="name side">
         <link name="${name}_wheel">
@@ -172,4 +176,28 @@
         <origin xyz="0.05 0 ${caster_radius - wheel_radius}" rpy="0 0 0"/>
     </joint>
+      <link name="camera_link">
+    <visual>
+      <geometry>
+        <box size="${cam_x} ${cam_y} ${cam_z}"/>
+      </geometry>
+      <material name="red"/>
+    </visual>
+    <collision>
+      <geometry>
+        <box size="${cam_x} ${cam_y} ${cam_z}"/>
+      </geometry>
+    </collision>
+    <inertial>
+      <mass value="${cam_mass}"/>
+      <inertia ixx="${cam_mass/12*(cam_y*cam_y+cam_z*cam_z)}" ixy="0" ixz="0"
+               iyy="${cam_mass/12*(cam_x*cam_x+cam_z*cam_z)}" iyz="0"
+               izz="${cam_mass/12*(cam_x*cam_x+cam_y*cam_y)}"/>
+    </inertial>
+  </link>
+  <joint name="camera_joint" type="fixed">
+    <parent link="base_link"/>
+    <child link="camera_link"/>
+    <origin xyz="0.06 0 0.05" rpy="0 0 0"/>
+  </joint>
         <!-- ===== Gazebo ===== -->
     <gazebo>
@@ -236,4 +264,24 @@
         </sensor>
     </gazebo>
+      <gazebo reference="camera_link">
+    <sensor name="camera_sensor" type="camera">
+      <always_on>true</always_on>
+      <update_rate>15</update_rate>
+      <topic>camera/image_raw</topic>
+      <gz_frame_id>camera_link</gz_frame_id>
+      <camera>
+        <horizontal_fov>1.047</horizontal_fov>
+        <image>
+          <width>640</width>
+          <height>480</height>
+          <format>R8G8B8</format>
+        </image>
+        <clip>
+          <near>0.05</near>
+          <far>10</far>
+        </clip>
+      </camera>
+    </sensor>
+    </gazebo>
     <gazebo reference="caster_front">
         <mu1>0.001</mu1>
